Commit message: Simple simulated urdf done

File: drone_ws/src/drone_description/urdf/drone.urdf.xacro (robot description, xacro)
@@ -6,7 +6,8 @@
 <!--        <xacro:include filename="$(find drone_description)/urdf/drone.gazebo.xacro" />-->
 <!--    </xacro:if>-->
+        <xacro:include filename="$(find drone_description)/urdf/macros.xacro" />
     <link name="base_link">
         <visual>
-            <origin xyz="0 0 0.1305"/>
+            <origin xyz="0 0 0"/>
             <geometry>
                 <mesh filename="package://drone_description/meshes/frame.stl"/>
@@ -25,31 +26,9 @@
         <parent link="base_link"/>
         <child link="landing_gear"/>
-        <origin rpy="0 0 0" xyz="0 0 0.1305"/>
+        <origin xyz="0 0 0" rpy="0 0 0"/>
     </joint>
-    <link name="motor">
-        <visual>
-            <origin xyz="-0.1591 -0.1591 0.1675"/>
-            <geometry>
-                <mesh filename="package://drone_description/meshes/motor.stl"/>
-            </geometry>
-        </visual>
-    </link>
-    <joint name="frame_to_motor" type="fixed">
-        <parent link="base_link"/>
-        <child link="motor"/>
-        <origin rpy="0 0 0" xyz="0 0 0"/>
-    </joint>
-    <link name="propeller">
-        <visual>
-            <origin xyz="-0.1591 -0.1591 0.19752"/>
-            <geometry>
-                <mesh filename="package://drone_description/meshes/propeller.stl"/>
-            </geometry>
-        </visual>
-    </link>
-    <joint name="motor_to_propeller" type="fixed">
-        <parent link="motor"/>
-        <child link="propeller"/>
-        <origin rpy="0 0 0" xyz="0 0 0"/>
-    </joint>
+    <xacro:motor_assembly number="1" x="0.1591" y="0.1591"/>
+    <xacro:motor_assembly number="2" x="-0.1591" y="0.1591"/>
+    <xacro:motor_assembly number="3" x="0.1591" y="-0.1591"/>
+    <xacro:motor_assembly number="4" x="-0.1591" y="-0.1591"/>
 </robot>

Commit message: Colision on the way

File: drone_ws/src/drone_description/urdf/drone.urdf.xacro (robot description, xacro)
@@ -2,5 +2,4 @@
 <robot name="drone" xmlns:xacro="http://www.ros.org/wiki/xacro">
     <xacro:arg name="use_sim" default="true" />
-<!--    <xacro:include filename="$(find drone_description)/urdf/core_structure.xacro" />-->
 <!--    <xacro:if value="$(arg use_sim)">-->
 <!--        <xacro:include filename="$(find drone_description)/urdf/drone.gazebo.xacro" />-->
@@ -14,4 +13,16 @@
             </geometry>
         </visual>
+        <collision>
+            <origin xyz="0 0 0.0115" rpy="0 0 0"/>
+            <geometry>
+                <box size="0.365 0.365 0.0575"/>
+            </geometry>
+        </collision>
+        <inertial>
+            <origin xyz="0.002 0  -0.009" rpy="0 0 0"/>
+            <mass value="0.803"/>
+            <inertia ixx="0.00565" ixy="0.000001" ixz="-0.000047"
+                    iyy="0.00602" iyz="-0.000002" izz="0.0113"/>
+        </inertial>
     </link>
     <link name="landing_gear">
@@ -22,4 +33,16 @@
             </geometry>
         </visual>
+        <collision>
+            <origin xyz="0 0 -0.065" rpy="0 0 0"/>
+            <geometry>
+                <box size="0.225 0.225 0.135"/>
+            </geometry>
+        </collision>
+        <inertial>
+            <origin xyz="0 0 -0.10" rpy="0 0 0"/>
+            <mass value="0.090"/>
+            <inertia ixx="0.00016" ixy="0" ixz="0"
+                    iyy="0.000641" iyz="0" izz="0.000769"/>
+        </inertial>
     </link>
     <joint name="frame_to_landing_gear" type="fixed">

File: drone_ws/src/drone_description/urdf/macros.xacro (robot description, xacro)
@@ -9,4 +9,16 @@
                 </geometry>
             </visual>
+            <colision>
+                <origin xyz="${x} ${y} 0.0385"/>
+                <geometry>
+                    <box size="0.225 0.225 0.135"/>
+                </geometry>
+            </colision>
+            <inertial>
+                <origin xyz="0 0 0" rpy="0 0 0"/>
+                <mass value="0.047"/>
+                <inertia ixx="5.7464844e-06" ixy="0.0" ixz="0.0"
+                        iyy="5.7464844e-06" iyz="0.0" izz="4.4429688e-06"/>
+            </inertial>
         </link>
         <joint name="frame_to_motor${number}" type="fixed">
@@ -22,4 +34,10 @@
                 </geometry>
             </visual>
+            <inertial>
+                <origin xyz="0 0 0" rpy="0 0 0"/>
+                <mass value="0.008"/>
+                <inertia ixx="1.00e-07" ixy="0.0" ixz="0.0"
+                        iyy="1.00e-07" iyz="0.0" izz="2.7526827e-05"/>
+            </inertial>
         </link>
         <joint name="motor_to_propeller${number}" type="fixed">

Commit message: Collision done

File: drone_ws/src/drone_description/urdf/drone.urdf.xacro (robot description, xacro)
@@ -20,5 +20,5 @@
         </collision>
         <inertial>
-            <origin xyz="0.002 0  -0.009" rpy="0 0 0"/>
+            <origin xyz="0 0 0" rpy="0 0 0"/>
             <mass value="0.803"/>
             <inertia ixx="0.00565" ixy="0.000001" ixz="-0.000047"

File: drone_ws/src/drone_description/urdf/macros.xacro (robot description, xacro)
@@ -9,10 +9,10 @@
                 </geometry>
             </visual>
-            <colision>
-                <origin xyz="${x} ${y} 0.0385"/>
+            <collision>
+                <origin xyz="0 0 0.0135" rpy="0 0 0"/>
                 <geometry>
-                    <box size="0.225 0.225 0.135"/>
+                    <box size="0.0225 0.0225 0.027"/>
                 </geometry>
-            </colision>
+            </collision>
             <inertial>
                 <origin xyz="0 0 0" rpy="0 0 0"/>
@@ -34,4 +34,10 @@
                 </geometry>
             </visual>
+            <collision>
+                <origin xyz="0 0 0" rpy="0 0 0"/>
+                <geometry>
+                    <box size="0.265 0.04 0.01"/>
+                </geometry>
+            </collision>
             <inertial>
                 <origin xyz="0 0 0" rpy="0 0 0"/>
