Commit message: Plugin plugged

File: drone_ws/src/drone_description/urdf/control/drone.gazebo.xacro (robot description, xacro)
@@ -2,5 +2,5 @@
 <robot name="drone" xmlns:xacro="http://www.ros.org/wiki/xacro">
     <gazebo>
-        <plugin filename="libteensy_emulator.so" name="TeensyEmulator">
+        <plugin filename="libTeensyEmulator.so" name="TeensyEmulator">
             <gain>150.0</gain>
         </plugin>

File: drone_ws/src/drone_description/urdf/robot/drone.urdf.xacro (robot description, xacro)
@@ -6,4 +6,10 @@
     </xacro:if>
     <xacro:include filename="$(find drone_description)/urdf/robot/macros.xacro" />
+    <link name="base_footprint"/>
+    <joint name="base_footprint_to_base_link" type="fixed">
+      <parent link="base_footprint"/>
+      <child link="base_link"/>
+      <origin xyz="0 0 0" rpy="0 0 0"/>
+    </joint>
     <link name="base_link">
         <visual>
