Commit message: Drone collored and ready to start flying

File: drone_ws/src/drone_description/urdf/robot/drone.urdf.xacro (robot description, xacro)
@@ -18,4 +18,7 @@
                 <mesh filename="package://drone_description/meshes/frame.stl"/>
             </geometry>
+            <material name="blue_body">
+                <color rgba="0.0 0.2 1.0 1.0"/>
+            </material>
         </visual>
         <collision>
@@ -38,4 +41,7 @@
                 <mesh filename="package://drone_description/meshes/landing_gear.stl"/>
             </geometry>
+            <material name="dark_gray">
+                <color rgba="0.15 0.15 0.15 1.0"/>
+            </material>
         </visual>
         <collision>

File: drone_ws/src/drone_description/urdf/robot/macros.xacro (robot description, xacro)
@@ -8,4 +8,7 @@
                     <mesh filename="package://drone_description/meshes/motor.stl"/>
                 </geometry>
+                <material name="bright_orange">
+                    <color rgba="1.0 0.45 0.05 1.0"/>
+                </material>
             </visual>
             <collision>
@@ -33,4 +36,7 @@
                     <mesh filename="package://drone_description/meshes/propeller.stl"/>
                 </geometry>
+                <material name="matte_black">
+                    <color rgba="0.05 0.05 0.05 1.0"/>
+                </material>
             </visual>
             <collision>
