Commit message: ekf filter working with IMU and GPS

File: ros2_ws/src/drone_description/urdf/robot/drone.urdf.xacro (robot description, xacro)
@@ -6,10 +6,4 @@
     </xacro:if>
     <xacro:include filename="$(find drone_description)/urdf/robot/macros.xacro" />
-    <link name="base_footprint"/>
-    <joint name="base_footprint_to_base_link" type="fixed">
-      <parent link="base_footprint"/>
-      <child link="base_link"/>
-      <origin xyz="0 0 0" rpy="0 0 0"/>
-    </joint>
     <link name="base_link">
         <visual>
